File: nfc.kicad_sch (KiCad schematic)
At the start: 0 parts

Commit message: Add hierarchical pins for Raspberry Pi connector
- Added hierarchical labels in raspberry_pn532.kicad_sch for connected J1 pins
- Added hierarchical pins on raspberry sheet in nfc.kicad_sch
- Pins: SDA, SCL, GPIO5, GPIO6, MISO, SCK, 5V, GND
Other:
- sheet raspberry_pn532 renamed raspberry (page 4)
- sheet raspberry (page 4) ports: added bidirectional, output; removed none
Changed lines of the file:
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@@
 			(color 0 0 0 0)
 		)
-		(property "Sheetname" "raspberry_pn532"
+		(property "Sheetname" "raspberry (page 4)"
 			(at 119.38 51.3584 0)
 			(show_name no)
@@
 			)
 		)
+	(pin output line
+		(at 168.91 63.50 0)
+		(length 2.54)
+		(name "SDA"
+			(effects
+				(font
+					(size 1.27 1.27)
+				)
+			)
+		)
+		(number "SDA"
+			(effects
+				(font
+					(size 1.27 1.27)
+				)
+			)
+		)
 	)
+	(pin output line
+		(at 168.91 66.04 0)
+		(length 2.54)
+		(name "SCL"
+			(effects
+				(font
+					(size 1.27 1.27)
+				)
+			)
+		)
+		(number "SCL"
+			(effects
+				(font
+					(size 1.27 1.27)
+				)
+			)
+		)
+	)
+	(pin output line
+		(at 168.91 73.66 0)
+		(length 2.54)
+		(name "GPIO5"
+			(effects
+				(font
+					(size 1.27 1.27)
+				)
+			)
+		)
+		(number "GPIO5"
+			(effects
+				(font
+					(size 1.27 1.27)
+				)
+			)
+		)
+	)
+	(pin output line
+		(at 168.91 76.20 0)
+		(length 2.54)
+		(name "GPIO6"
+			(effects
+				(font
+					(size 1.27 1.27)
+				)
+			)
+		)
+		(number "GPIO6"
+			(effects
+				(font
+					(size 1.27 1.27)
+				)
+			)
+		)
+	)
+	(pin output line
+		(at 168.91 86.36 0)
+		(length 2.54)
+		(name "MISO"
+			(effects
+				(font
+					(size 1.27 1.27)
+				)
+			)
+		)
+		(number "MISO"
+			(effects
+				(font
+					(size 1.27 1.27)
+				)
+			)
+		)
+	)
+	(pin output line
+		(at 168.91 91.44 0)
+		(length 2.54)
+		(name "SCK"
+			(effects
+				(font
+					(size 1.27 1.27)
+				)
+			)
+		)
+		(number "SCK"
+			(effects
+				(font
+					(size 1.27 1.27)
+				)
+			)
+		)
+	)
+	(pin bidirectional line
+		(at 127.00 52.07 270)
+		(length 2.54)
+		(name "5V"
+			(effects
+				(font
+					(size 1.27 1.27)
+				)
+			)
+		)
+		(number "5V"
+			(effects
+				(font
+					(size 1.27 1.27)
+				)
+			)
+		)
+	)
+	(pin bidirectional line
+		(at 101.60 90.17 90)
+		(length 2.54)
+		(name "GND"
+			(effects
+				(font
+					(size 1.27 1.27)
+				)
+			)
+		)
+		(number "GND"
+			(effects
+				(font
+					(size 1.27 1.27)
+				)
+			)
+		)
+	)
+)
 	(sheet
 		(at 210.82 49.53)
