File: nfc.kicad_sch (KiCad schematic)
At the start: 0 parts

Commit message: Fix hierarchical pin format: (pin "name" type) instead of (pin type (name...))
Other:
- sheet raspberry (page 4) ports: added +5, +5V, +5_1, 1V8, 3V3, BT_ON, CORE, GCLK0/GPIO4, GCLK1/GPIO5, GCLK2/GPIO6, GPIO14/TXD, GPIO15/RXD, GPIO16, GPIO17, GPIO18/PWM0, GPIO19/MISO1, GPIO20/MOSI1, GPIO21/SCLK1, GPIO22, GPIO23, GPIO24, GPIO25, GPIO26, GPIO27, GPIO4, ID_SC/GPIO1, ID_SD/GPIO0, MISO0/GPIO9, MOSI0/GPIO10, OTG, PWM0/GPIO12, PWM1/GPIO13, RUN, SCL/GPIO3, SCLK0/GPIO11, SDA/GPIO2, SD_CLK, SD_CMD, SD_DAT0, SD_DAT1, SD_DAT2, SD_DAT3, SD__1, SD__2, SD__3, STATUS_LED, TV, USB_DM, USB_DP, WL_ON, ~{CE0}/GPIO8, ~{CE1}/GPIO7; removed bidirectional
