File: oled.kicad_sch (KiCad schematic)
At the start: 7 parts, among them J2 OledSpiST1306, J3 OledSpiST7789

Commit message: Add hierarchical labels/pins across all sheets, fix DiscoveryAnalog3 rename, PCB 99x99mm rounded corners
- nfc_rpi.kicad_sch: 19 hierarchical pins on PN532 sheet
- pn532.kicad_sch: 22 hierarchical labels with _PN532 suffix
- raspberry_pn532.kicad_sch: 68 hierarchical labels for J1
- nfc.kicad_sch: 54 signal pins on Raspberry sheet, power pins removed
- switch.kicad_sch: 8 switch+resistor circuits with hierarchical labels
- oled.kicad_sch: 7 hierarchical labels
- DiscoveryAnalog3.kicad_sch: 26 hierarchical labels for J4 connector
- nfc_rpi.kicad_pcb: 99x99mm board outline with 5mm rounded corners (gr_line + gr_arc)
Parts:
- removed C10, C8, C9: 100n, Capacitor_SMD:C_0603_1608Metric, symbol Device:C
Connections:
- net +3V3: now also J3.2 (Pin_2)
- net +5V: no longer J3.2 (Pin_2)
- net SCL_OLED_RPI renamed SCL_OLED
- net SDA_OLED_RPI renamed SDA_OLED
