File: switch.kicad_sch (KiCad schematic)
At the start: 16 parts, among them SW1 mclr, SW5 mclr

Commit message: Add hierarchical labels/pins across all sheets, fix DiscoveryAnalog3 rename, PCB 99x99mm rounded corners
- nfc_rpi.kicad_sch: 19 hierarchical pins on PN532 sheet
- pn532.kicad_sch: 22 hierarchical labels with _PN532 suffix
- raspberry_pn532.kicad_sch: 68 hierarchical labels for J1
- nfc.kicad_sch: 54 signal pins on Raspberry sheet, power pins removed
- switch.kicad_sch: 8 switch+resistor circuits with hierarchical labels
- oled.kicad_sch: 7 hierarchical labels
- DiscoveryAnalog3.kicad_sch: 26 hierarchical labels for J4 connector
- nfc_rpi.kicad_pcb: 99x99mm board outline with 5mm rounded corners (gr_line + gr_arc)
Parts:
- removed R10, R9: (no value), Resistor_SMD:R_0805_2012Metric, symbol Device:R_US
- removed SW1: mclr, Button_Switch_SMD:SW_Push_1P1T_NO_CK_KSC6xxJ, symbol Switch:SW_Push_Dual_x2
- removed SW7, SW8: (no value), Button_Switch_SMD:SW_Push_1P1T_NO_CK_KSC6xxJ, symbol Switch:SW_Push_Dual_x2
- added SW4: (no value), Button_Switch_SMD:SW_Push_1P1T_NO_CK_KSC6xxJ, symbol Switch:SW_Push_Dual_x2
- SW5: value mclr -> (none)
- renumbered SW4 to SW1
Connections:
- net GND: now also SW4.1 (C)
- net at R3.2: now also SW1.2 (D)
- net at R6.2: now also SW4.2 (D); no longer SW1.2 (D)
- net GPIO24 renamed sw4
- net GPIO25 renamed sw3
- net GPIO26 renamed sw2
- net GPIO27 renamed sw1
- net GPIO28 renamed sw5
- net GPIO29 renamed sw6
Other:
- moved on the sheet: SW1A
